File: ESP-TC-PROG.kicad_pcb (KiCad board)
At the start: 2 copper layers, 40 x 18 mm, 22 parts, among them J1 USB, J2 TC, J3 PINH, Q1 AO3400A, Q2 AO3400A, Q3 AO3400A, U1 USBLC6-4, U2 CH340G, Y1 12Mhz

Commit message: finalized silk
Parts:
- moved R4 24.2 mm to (121.3, 101.3), turned to 90 degrees
- moved C2 22.2 mm to (110.9, 96.9), turned to 90 degrees
- moved R5 20.0 mm to (121.7, 97.2), turned to 180 degrees
- moved C3 18.5 mm to (119.3, 93.9), turned to 90 degrees
- moved Y1 14.6 mm to (111.2, 103.5)
- moved C4 14.3 mm to (108.5, 104.2)
- moved C5 12.6 mm to (114.3, 105.8), turned to 180 degrees
- moved C1 7.07 mm to (117.5, 94.2), turned to 180 degrees
- moved J3 6.05 mm to (135.4, 100.0)
- moved Q3 5.85 mm to (122.7, 103.0), turned to 180 degrees
- moved J2 5.70 mm to (129.3, 100.0), turned to 180 degrees
- moved Q1 5.44 mm to (122.6, 99.4)
- moved Q2 5.28 mm to (122.5, 95.0)
- moved R6 5.19 mm to (120.9, 93.5)
- moved R1 1.36 mm to (108.6, 98.3)
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Other:
- board size 40 x 18 mm -> 38.2 x 16.1 mm
- board text added: "EN"
- board text added: "ESP-TC-Prog."
- board text added: "GND"
- board text added: "IO0"
- board text added: "PWR"
- board text added: "RXD"
- board text added: "TXD"
- board text added: "nIO0"

Commit message: export greber
Parts:
- Q3: value AO3400A -> AO3401A
- moved Q3 7.98 mm to (122.5, 95.0), turned to 90 degrees
- moved R5 3.43 mm to (121.7, 100.6)
- moved Q1 3.42 mm to (122.6, 102.8)
- moved Q2 3.42 mm to (122.5, 98.4)
- moved R4 2.37 mm to (123.6, 100.6), turned to 0 degrees
- moved R1 0.15 mm to (108.6, 98.2)
Connections:
- Q3 pad 2: GND -> V3
Routing:
- net VBUS: track 0.00 -> 32.3 mm, vias 0 -> 5
- net TXD: track 0.00 -> 23.8 mm, vias 0 -> 1
- net RXD: track 0.00 -> 23.5 mm, vias 0 -> 1
- net nIO0: track 0.00 -> 23.5 mm, vias 0 -> 1
- net IO0: track 0.00 -> 21.6 mm
- net V3: track 0.00 -> 18.6 mm, vias 0 -> 2
- net EN: track 0.00 -> 18.4 mm, vias 0 -> 2
- net D+: track 0.00 -> 13.2 mm, vias 0 -> 2
- net D-: track 0.00 -> 12.8 mm
- net Net-(R4-Pad2): track 0.00 -> 12.7 mm
- net GND: track 0.00 -> 10.3 mm, vias 0 -> 35
- net Net-(C4-Pad2): track 0.00 -> 6.70 mm, vias 0 -> 2
- net Net-(R5-Pad2): track 0.00 -> 3.93 mm
- net Net-(C5-Pad1): track 0.00 -> 3.72 mm
- net Net-(Q1-Pad2): track 0.00 -> 2.85 mm
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- added copper zone on B.Cu, net GND
- added copper zone on F.Cu, net GND
Other:
- board size 38.2 x 16.1 mm -> 37.6 x 16.1 mm
- net class Default: trace_width 0.25 -> 0.2; via_dia 0.8 -> 0.6
- rule pad_to_mask_clearance: 0.051 -> 0
- board text added: "Design by: @JanHenrikH @FauthNiklas"
- board text added: "v1.0"

Commit message: update
Parts:
- moved C4 6.47 mm to (114.8, 105.8), turned to 0 degrees
- moved C5 6.05 mm to (108.5, 104.2), turned to 270 degrees
- turned Y1 to 0 degrees
Connections:
- Y1 pad 1: GND -> Net-(C5-Pad1)
- Y1 pad 2: Net-(C4-Pad2) -> GND
- Y1 pad 3: GND -> Net-(C4-Pad2)
- Y1 pad 4: Net-(C5-Pad1) -> GND
Routing:
- net GND: track 10.3 -> 16.0 mm, vias 35 -> 36
- net Net-(C5-Pad1): track 3.72 -> 7.06 mm
- net Net-(C4-Pad2): track 6.70 -> 6.29 mm, vias 2 -> 0
Changed lines of the file:
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@@
     (thickness 1.6)
     (drawings 34)
-    (tracks 241)
+    (tracks 246)
     (zones 0)
     (modules 22)
@@
   )
   (module Crystal:Crystal_SMD_3225-4Pin_3.2x2.5mm (layer F.Cu)
-    (at 111.2 103.5 180)
+    (at 111.19 103.5)
     (descr "SMD Crystal SERIES SMD3225/4 http://www.txccrystal.com/images/pdf/7m-accuracy.pdf, 3.2x2.5mm^2 package")
     (tags "SMD SMT crystal")
@@
       (effects (font (size 0.5 0.5) (thickness 0.1)))
     )
-    (pad 4 smd rect (at -1.1 -0.85 180) (size 1.4 1.2) (layers F.Cu F.Paste F.Mask)
+    (pad 4 smd rect (at -1.1 -0.85) (size 1.4 1.2) (layers F.Cu F.Paste F.Mask)
+      (net 1 GND))
+    (pad 3 smd rect (at 1.1 -0.85) (size 1.4 1.2) (layers F.Cu F.Paste F.Mask)
+      (net 3 "Net-(C4-Pad2)"))
+    (pad 2 smd rect (at 1.1 0.85) (size 1.4 1.2) (layers F.Cu F.Paste F.Mask)
+      (net 1 GND))
+    (pad 1 smd rect (at -1.1 0.85) (size 1.4 1.2) (layers F.Cu F.Paste F.Mask)
       (net 4 "Net-(C5-Pad1)"))
-    (pad 3 smd rect (at 1.1 -0.85 180) (size 1.4 1.2) (layers F.Cu F.Paste F.Mask)
-      (net 1 GND))
-    (pad 2 smd rect (at 1.1 0.85 180) (size 1.4 1.2) (layers F.Cu F.Paste F.Mask)
-      (net 3 "Net-(C4-Pad2)"))
-    (pad 1 smd rect (at -1.1 0.85 180) (size 1.4 1.2) (layers F.Cu F.Paste F.Mask)
-      (net 1 GND))
     (model ${KISYS3DMOD}/Crystal.3dshapes/Crystal_SMD_3225-4Pin_3.2x2.5mm.wrl
       (at (xyz 0 0 0))
@@
   )
   (module otter:C_0402 (layer F.Cu)
-    (at 114.3 105.8 180)
+    (at 108.46 104.23 270)
     (descr "Capacitor 0402")
     (tags "C Capacitor 0402")
     (attr smd)
-    (fp_text reference C5 (at 1.4 0) (layer F.SilkS)
-      (effects (font (size 0.5 0.5) (thickness 0.1)))
-    )
-    (fp_text value 22p (at 0 -1.325) (layer F.Fab) hide
+    (fp_text reference C5 (at 1.4 0 90) (layer F.SilkS)
+      (effects (font (size 0.5 0.5) (thickness 0.1)))
+    )
+    (fp_text value 22p (at 0 -1.325 90) (layer F.Fab) hide
       (effects (font (size 1 1) (thickness 0.15)))
     )
     (fp_line (start 0 0.15) (end 0 -0.15) (layer F.SilkS) (width 0.12))
-    (pad 2 smd rect (at 0.47 0 180) (size 0.5 0.6) (layers F.Cu F.Paste F.Mask)
-      (net 1 GND))
-    (pad 1 smd rect (at -0.47 0 180) (size 0.5 0.6) (layers F.Cu F.Paste F.Mask)
+    (pad 2 smd rect (at 0.47 0 270) (size 0.5 0.6) (layers F.Cu F.Paste F.Mask)
+      (net 1 GND))
+    (pad 1 smd rect (at -0.47 0 270) (size 0.5 0.6) (layers F.Cu F.Paste F.Mask)
       (net 4 "Net-(C5-Pad1)"))
     (model ${KISYS3DMOD}/Capacitor_SMD.3dshapes/C_0402_1005Metric.step
@@
   )
   (module otter:C_0402 (layer F.Cu)
-    (at 108.5 104.23 90)
+    (at 114.78 105.79)
     (descr "Capacitor 0402")
     (tags "C Capacitor 0402")
     (attr smd)
-    (fp_text reference C4 (at -0.82 -0.95 180) (layer F.SilkS)
-      (effects (font (size 0.5 0.5) (thickness 0.1)))
-    )
-    (fp_text value 22p (at 0 -1.325 90) (layer F.Fab) hide
+    (fp_text reference C4 (at -0.82 -0.95 270) (layer F.SilkS)
+      (effects (font (size 0.5 0.5) (thickness 0.1)))
+    )
+    (fp_text value 22p (at 0 -1.325) (layer F.Fab) hide
       (effects (font (size 1 1) (thickness 0.15)))
     )
     (fp_line (start 0 0.15) (end 0 -0.15) (layer F.SilkS) (width 0.12))
-    (pad 2 smd rect (at 0.47 0 90) (size 0.5 0.6) (layers F.Cu F.Paste F.Mask)
+    (pad 2 smd rect (at 0.47 0) (size 0.5 0.6) (layers F.Cu F.Paste F.Mask)
       (net 3 "Net-(C4-Pad2)"))
-    (pad 1 smd rect (at -0.47 0 90) (size 0.5 0.6) (layers F.Cu F.Paste F.Mask)
+    (pad 1 smd rect (at -0.47 0) (size 0.5 0.6) (layers F.Cu F.Paste F.Mask)
       (net 1 GND))
     (model ${KISYS3DMOD}/Capacitor_SMD.3dshapes/C_0402_1005Metric.step
@@
   (gr_line (start 100 90) (end 100 110) (layer Eco1.User) (width 0.15))
   (gr_line (start 93.95 100) (end 133.95 100) (layer Eco1.User) (width 0.15))
-  (segment (start 108.07 103.2) (end 107 103.2) (width 0.2) (layer F.Cu) (net 1))
-  (segment (start 108.5 102.77) (end 108.07 103.2) (width 0.2) (layer F.Cu) (net 1))
   (via (at 109.1 101.1) (size 0.6) (drill 0.4) (layers F.Cu B.Cu) (net 1))
-  (segment (start 112.2 102.65) (end 111.55 103.3) (width 0.3) (layer F.Cu) (net 1))
-  (segment (start 111.55 103.3) (end 111.3 103.3) (width 0.3) (layer F.Cu) (net 1))
-  (segment (start 110.9 101.35) (end 110.9 100.9) (width 0.3) (layer F.Cu) (net 1))
-  (segment (start 112.2 102.65) (end 110.9 101.35) (width 0.3) (layer F.Cu) (net 1))
-  (segment (start 112.3 102.65) (end 112.2 102.65) (width 0.3) (layer F.Cu) (net 1))
-  (via (at 112.8 105.6) (size 0.6) (drill 0.4) (layers F.Cu B.Cu) (net 1))
-  (via (at 111.6 105.5) (size 0.6) (drill 0.4) (layers F.Cu B.Cu) (net 1))
-  (segment (start 109.75 104.7) (end 110.1 104.35) (width 0.3) (layer F.Cu) (net 1))
-  (segment (start 109.1 104.7) (end 109.1 105) (width 0.3) (layer F.Cu) (net 1))
-  (segment (start 108.5 104.7) (end 109.1 104.7) (width 0.3) (layer F.Cu) (net 1))
-  (segment (start 109.1 104.7) (end 109.75 104.7) (width 0.3) (layer F.Cu) (net 1))
   (segment (start 107 103.405) (end 106.085 104.32) (width 0.3) (layer F.Cu) (net 1))
   (segment (start 107 103.2) (end 107 103.405) (width 0.3) (layer F.Cu) (net 1))
@@
   (via (at 133.9 107.1) (size 0.6) (drill 0.4) (layers F.Cu B.Cu) (net 1))
   (via (at 124.35 107.1) (size 0.6) (drill 0.4) (layers F.Cu B.Cu) (net 1))
+  (segment (start 108.07 103.2) (end 107 103.2) (width 0.2) (layer F.Cu) (net 1))
+  (segment (start 108.5 102.77) (end 108.07 103.2) (width 0.2) (layer F.Cu) (net 1))
+  (segment (start 107.715 104.7) (end 108.04999 104.7) (width 0.2) (layer F.Cu) (net 1))
+  (segment (start 106.085 104.32) (end 107.335 104.32) (width 0.2) (layer F.Cu) (net 1))
+  (segment (start 107.335 104.32) (end 107.715 104.7) (width 0.2) (layer F.Cu) (net 1))
+  (segment (start 106.465 104.7) (end 106.085 104.32) (width 0.2) (layer F.Cu) (net 1))
+  (segment (start 108.46 104.7) (end 106.465 104.7) (width 0.2) (layer F.Cu) (net 1))
+  (segment (start 110.9 101.84) (end 110.09 102.65) (width 0.2) (layer F.Cu) (net 1))
+  (segment (start 110.9 100.9) (end 110.9 101.84) (width 0.2) (layer F.Cu) (net 1))
+  (segment (start 108.62 102.65) (end 108.5 102.77) (width 0.2) (layer F.Cu) (net 1))
+  (segment (start 110.09 102.65) (end 108.62 102.65) (width 0.2) (layer F.Cu) (net 1))
+  (segment (start 110.19 102.65) (end 110.09 102.65) (width 0.2) (layer F.Cu) (net 1))
+  (segment (start 111.89 104.35) (end 111.37 103.83) (width 0.2) (layer F.Cu) (net 1))
+  (segment (start 112.29 104.35) (end 111.89 104.35) (width 0.2) (layer F.Cu) (net 1))
+  (segment (start 111.37 103.83) (end 110.19 102.65) (width 0.2) (layer F.Cu) (net 1))
+  (via (at 111.37 103.83) (size 0.6) (drill 0.4) (layers F.Cu B.Cu) (net 1))
+  (via (at 113.37 105.84) (size 0.6) (drill 0.4) (layers F.Cu B.Cu) (net 1))
+  (via (at 116.53 105.93) (size 0.6) (drill 0.4) (layers F.Cu B.Cu) (net 1))
   (segment (start 110.9 98.7) (end 110.9 97.37) (width 0.4) (layer F.Cu) (net 2))
   (segment (start 119.475 94.495) (end 119.35 94.37) (width 0.4) (layer F.Cu) (net 2))
@@
   (segment (start 111.75 98.23) (end 111.75 97.35) (width 0.4) (layer B.Cu) (net 2))
   (segment (start 111.81 98.29) (end 111.75 98.23) (width 0.4) (layer B.Cu) (net 2))
-  (via (at 113.62 102.81) (size 0.6) (drill 0.4) (layers F.Cu B.Cu) (net 3))
-  (segment (start 114.525 103.175) (end 113.985 103.175) (width 0.2) (layer F.Cu) (net 3))
-  (segment (start 113.985 103.175) (end 113.62 102.81) (width 0.2) (layer F.Cu) (net 3))
-  (via (at 110.96 102.71) (size 0.6) (drill 0.4) (layers F.Cu B.Cu) (net 3))
-  (segment (start 113.62 102.81) (end 111.06 102.81) (width 0.2) (layer B.Cu) (net 3))
-  (segment (start 111.06 102.81) (end 110.96 102.71) (width 0.2) (layer B.Cu) (net 3))
-  (segment (start 110.16 102.71) (end 110.1 102.65) (width 0.2) (layer F.Cu) (net 3))
-  (segment (start 110.96 102.71) (end 110.16 102.71) (width 0.2) (layer F.Cu) (net 3))
-  (segment (start 110 102.65) (end 110.1 102.65) (width 0.2) (layer F.Cu) (net 3))
-  (segment (start 108.89 103.76) (end 110 102.65) (width 0.2) (layer F.Cu) (net 3))
-  (segment (start 108.5 103.76) (end 108.89 103.76) (width 0.2) (layer F.Cu) (net 3))
-  (segment (start 114.43 104.35) (end 114.525 104.445) (width 0.2) (layer F.Cu) (net 4))
-  (segment (start 112.3 104.35) (end 114.43 104.35) (width 0.2) (layer F.Cu) (net 4))
-  (segment (start 114.77 104.69) (end 114.525 104.445) (width 0.2) (layer F.Cu) (net 4))
-  (segment (start 114.77 105.8) (end 114.77 104.69) (width 0.2) (layer F.Cu) (net 4))
+  (segment (start 112.815 103.175) (end 112.29 102.65) (width 0.2) (layer F.Cu) (net 3))
+  (segment (start 114.525 103.175) (end 112.815 103.175) (width 0.2) (layer F.Cu) (net 3))
+  (segment (start 115.85 105.1) (end 115.25 105.7) (width 0.2) (layer F.Cu) (net 3))
+  (segment (start 114.525 103.175) (end 115.255 103.175) (width 0.2) (layer F.Cu) (net 3))
+  (segment (start 115.25 105.7) (end 115.25 105.79) (width 0.2) (layer F.Cu) (net 3))
+  (segment (start 115.85 103.77) (end 115.85 105.1) (width 0.2) (layer F.Cu) (net 3))
+  (segment (start 115.255 103.175) (end 115.85 103.77) (width 0.2) (layer F.Cu) (net 3))
+  (segment (start 109.5 103.76) (end 108.46 103.76) (width 0.2) (layer F.Cu) (net 4))
+  (segment (start 110.09 104.35) (end 109.5 103.76) (width 0.2) (layer F.Cu) (net 4))
+  (segment (start 110.09 104.39) (end 110.09 104.35) (width 0.2) (layer F.Cu) (net 4))
+  (segment (start 113.730001 105.239999) (end 113.081999 105.239999) (width 0.2) (layer F.Cu) (net 4))
+  (segment (start 110.98 105.28) (end 110.09 104.39) (width 0.2) (layer F.Cu) (net 4))
+  (segment (start 114.525 104.445) (end 113.730001 105.239999) (width 0.2) (layer F.Cu) (net 4))
+  (segment (start 113.041998 105.28) (end 110.98 105.28) (width 0.2) (layer F.Cu) (net 4))
+  (segment (start 113.081999 105.239999) (end 113.041998 105.28) (width 0.2) (layer F.Cu) (net 4))
   (segment (start 112.6 98.02) (end 112.6 97.37) (width 0.4) (layer F.Cu) (net 5))
   (segment (start 112.6 98.815) (end 112.6 98.02) (width 0.4) (layer F.Cu) (net 5))
