File: ESP-TC-PROG.sch (KiCad schematic (older format))
At the start: 22 parts, among them J1 USB, J2 TC, J3 PINH, Q1 AO3400A, Q2 AO3400A, Q3 AO3400A, U1 USBLC6-4, U2 CH340G, Y1 12Mhz

Commit message: export greber
Parts:
- removed Q3: AO3400A, Package_TO_SOT_SMD:SOT-23, symbol Transistor_FET:2N7002
- added Q3: AO3401A, Package_TO_SOT_SMD:SOT-23, symbol Transistor_FET:AO3401A
Connections:
- net IO0: now also Q3.1 (G)
- net V3: now also Q3.2 (S)
- net nIO0: now also Q3.3 (D)
Changed lines of the file:
@@
 Wire Wire Line
 	7650 3700 7750 3700
-Text GLabel 8050 3500 1    50   Input ~ 0
+Text GLabel 8050 3900 3    50   Input ~ 0
 nIO0
-$Comp
-L power:GND #PWR0119
-U 1 1 5E80356D
-P 8050 3900
-F 0 "#PWR0119" H 8050 3650 50  0001 C CNN
-F 1 "GND" H 8055 3727 50  0000 C CNN
-F 2 "" H 8050 3900 50  0001 C CNN
-F 3 "" H 8050 3900 50  0001 C CNN
-	1    8050 3900
-	1    0    0    -1
-$EndComp
 Text GLabel 5350 2350 1    50   Input ~ 0
 V3
@@
 $EndComp
 Connection ~ 7350 3450
-$Comp
-L Transistor_FET:2N7002 Q3
-U 1 1 5E84CC24
-P 7950 3700
-F 0 "Q3" H 8155 3746 50  0000 L CNN
-F 1 "AO3400A" H 8155 3655 50  0000 L CNN
-F 2 "Package_TO_SOT_SMD:SOT-23" H 8150 3625 50  0001 L CIN
-F 3 "https://www.fairchildsemi.com/datasheets/2N/2N7002.pdf" H 7950 3700 50  0001 L CNN
-	1    7950 3700
-	1    0    0    -1
-$EndComp
 $Comp
 L Device:LED D1
@@
 	5300 3500 5300 3550
 Connection ~ 5300 3550
+$Comp
+L Transistor_FET:AO3401A Q3
+U 1 1 5E916262
+P 7950 3700
+F 0 "Q3" H 8155 3654 50  0000 L CNN
+F 1 "AO3401A" H 8155 3745 50  0000 L CNN
+F 2 "Package_TO_SOT_SMD:SOT-23" H 8150 3625 50  0001 L CIN
+F 3 "http://www.aosmd.com/pdfs/datasheet/AO3401A.pdf" H 7950 3700 50  0001 L CNN
+	1    7950 3700
+	1    0    0    1
+$EndComp
+Text GLabel 8050 3500 1    50   Input ~ 0
+V3
 $EndSCHEMATC

Commit message: update
Connections:
- net GND: now also Y1.2, Y1.4; no longer Y1.1, Y1.3
- net at C4.2, U2.7 (XI): now also Y1.3; no longer Y1.2
- net at C5.1, U2.8 (XO): now also Y1.1; no longer Y1.4
Other:
- moved on the sheet: C4, C5
Changed lines of the file:
@@
 L power:GND #PWR0114
 U 1 1 5E7C39CC
-P 5150 3300
-F 0 "#PWR0114" H 5150 3050 50  0001 C CNN
-F 1 "GND" V 5155 3172 50  0000 R CNN
-F 2 "" H 5150 3300 50  0001 C CNN
-F 3 "" H 5150 3300 50  0001 C CNN
-	1    5150 3300
+P 5100 3300
+F 0 "#PWR0114" H 5100 3050 50  0001 C CNN
+F 1 "GND" V 5105 3172 50  0000 R CNN
+F 2 "" H 5100 3300 50  0001 C CNN
+F 3 "" H 5100 3300 50  0001 C CNN
+	1    5100 3300
 	0    1    1    0
 $EndComp
@@
 L Device:C_Small C5
 U 1 1 5E7C58F5
-P 5200 3550
-F 0 "C5" V 5337 3550 50  0000 C CNN
-F 1 "22p" V 5428 3550 50  0000 C CNN
-F 2 "otter:C_0402" H 5200 3550 50  0001 C CNN
-F 3 "~" H 5200 3550 50  0001 C CNN
-	1    5200 3550
+P 5200 3500
+F 0 "C5" V 5337 3500 50  0000 C CNN
+F 1 "22p" V 5428 3500 50  0000 C CNN
+F 2 "otter:C_0402" H 5200 3500 50  0001 C CNN
+F 3 "~" H 5200 3500 50  0001 C CNN
+	1    5200 3500
 	0    1    1    0
 $EndComp
@@
 L Device:C_Small C4
 U 1 1 5E7C6116
-P 5200 3050
-F 0 "C4" V 5429 3050 50  0000 C CNN
-F 1 "22p" V 5338 3050 50  0000 C CNN
-F 2 "otter:C_0402" H 5200 3050 50  0001 C CNN
-F 3 "~" H 5200 3050 50  0001 C CNN
-	1    5200 3050
+P 5200 3100
+F 0 "C4" V 5429 3100 50  0000 C CNN
+F 1 "22p" V 5338 3100 50  0000 C CNN
+F 2 "otter:C_0402" H 5200 3100 50  0001 C CNN
+F 3 "~" H 5200 3100 50  0001 C CNN
+	1    5200 3100
 	0    -1   -1   0
 $EndComp
@@
 L power:GND #PWR0115
 U 1 1 5E7C9132
-P 5100 3050
-F 0 "#PWR0115" H 5100 2800 50  0001 C CNN
-F 1 "GND" V 5105 2922 50  0000 R CNN
-F 2 "" H 5100 3050 50  0001 C CNN
-F 3 "" H 5100 3050 50  0001 C CNN
-	1    5100 3050
+P 5100 3100
+F 0 "#PWR0115" H 5100 2850 50  0001 C CNN
+F 1 "GND" V 5105 2972 50  0000 R CNN
+F 2 "" H 5100 3100 50  0001 C CNN
+F 3 "" H 5100 3100 50  0001 C CNN
+	1    5100 3100
 	0    1    1    0
 $EndComp
@@
 L power:GND #PWR0116
 U 1 1 5E7C9A53
-P 5100 3550
-F 0 "#PWR0116" H 5100 3300 50  0001 C CNN
-F 1 "GND" V 5105 3422 50  0000 R CNN
-F 2 "" H 5100 3550 50  0001 C CNN
-F 3 "" H 5100 3550 50  0001 C CNN
-	1    5100 3550
+P 5100 3500
+F 0 "#PWR0116" H 5100 3250 50  0001 C CNN
+F 1 "GND" V 5105 3372 50  0000 R CNN
+F 2 "" H 5100 3500 50  0001 C CNN
+F 3 "" H 5100 3500 50  0001 C CNN
+	1    5100 3500
 	0    1    1    0
 $EndComp
@@
 F 3 "~" H 5300 3300 50  0001 C CNN
 	1    5300 3300
-	1    0    0    -1
-$EndComp
-Wire Wire Line
-	5300 3550 5600 3550
-Wire Wire Line
-	5600 3050 5300 3050
-Wire Wire Line
-	5600 3050 5600 3200
-Wire Wire Line
-	5600 3400 5600 3550
+	0    -1   -1   0
+$EndComp
+Wire Wire Line
+	5300 3500 5600 3500
+Wire Wire Line
+	5600 3100 5300 3100
+Wire Wire Line
+	5600 3400 5600 3500
 $Comp
 L power:GND #PWR0124
 U 1 1 5E887A23
-P 5450 3300
-F 0 "#PWR0124" H 5450 3050 50  0001 C CNN
-F 1 "GND" V 5455 3172 50  0000 R CNN
-F 2 "" H 5450 3300 50  0001 C CNN
-F 3 "" H 5450 3300 50  0001 C CNN
-	1    5450 3300
-	0    -1   -1   0
-$EndComp
-Wire Wire Line
-	5300 3100 5300 3050
-Connection ~ 5300 3050
-Wire Wire Line
-	5300 3500 5300 3550
-Connection ~ 5300 3550
+P 5500 3300
+F 0 "#PWR0124" H 5500 3050 50  0001 C CNN
+F 1 "GND" V 5505 3172 50  0000 R CNN
+F 2 "" H 5500 3300 50  0001 C CNN
+F 3 "" H 5500 3300 50  0001 C CNN
+	1    5500 3300
+	0    -1   -1   0
+$EndComp
+Wire Wire Line
+	5300 3150 5300 3100
+Connection ~ 5300 3100
+Wire Wire Line
+	5300 3450 5300 3500
+Connection ~ 5300 3500
 $Comp
 L Transistor_FET:AO3401A Q3
@@
 Text GLabel 8050 3500 1    50   Input ~ 0
 V3
+Wire Wire Line
+	5600 3100 5600 3200
 $EndSCHEMATC
