File: ESP-TC-PROG.kicad_sch (KiCad schematic)
At the start: 22 parts, among them J1 USB, J2 TC, J3 PINH, Q1 AO3400A, Q2 AO3400A, Q3 AO3401A, U1 USBLC6-4, U2 CH340G, Y1 12Mhz

Commit message: updated to v1.2.1
Parts:
- removed Q1, Q2: AO3400A, Package_TO_SOT_SMD:SOT-23, symbol Transistor_FET:2N7002
- removed Q3: AO3401A, Package_TO_SOT_SMD:SOT-23, symbol Transistor_FET:AO3401A
- added Q1, Q2: S8050-J3Y, Package_TO_SOT_SMD:SOT-23, symbol caffeinated-labs:S8050-J3Y
- added R7: 5k1, otter:R_0402, symbol Device:R_Small
- C1: value 10µ -> 4u7; footprint otter:C_0603 -> otter:C_0805
- C2, C3, C6: value 0.1µ -> 100n
- R6: value 100k -> 5k1
- U2: value CH340G -> CH340G/C
Connections:
- net EN: now also R6.2, Q1.3 (C)
- net IO0: now also Q2.3 (C), R7.1; no longer R6.2
- net V3: now also R7.2
- net at R4.2, U2.13 (~{DTR}): now also Q2.2 (E)
- net at R5.2, U2.14 (~{RTS}): now also Q1.2 (E)
- net at R4.1: now also Q1.1 (B)
- net at R5.1: now also Q2.1 (B)
- net nIO0: no longer names the net of J3.1 (Pin_1)
Other:
- moved on the sheet: R4, R5
